File: Licencjat_v1.kicad_pcb (KiCad board)
At the start: 2 copper layers, 85 x 65 mm, 73 parts, among them J1 PV_IN_1, J10 SERIAL, J2 PV_IN_2, J3 AHT20 + BMP280, J4 VEML7700, J5 ADDITIONAL I2C, J6 RF_TRANSMITTER, J7 AVR-ISP-6, J8 GEIGER, J9 1_WIRE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

Commit message: Adjust values
Parts:
- C14: value 1u -> 100p
- C3: value C_Small -> 100n
- C4: value C_Small -> 10u
- Q11, Q4, Q5, Q6: value AO3400A -> BSS138
- Q2: value BC846 -> BC847
- R1, R2: value R_Small -> 1k
- R10, R7: value R_Small -> 100k
- R11, R8: value R_Small -> 1M
- R17: value 47k -> 470k
- R4: value 10k -> 240k
Changed lines of the file:
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@@
 			)
 		)
-		(property "Value" "R_Small"
+		(property "Value" "1k"
 			(at 0 -1.83 90)
 			(layer "B.Fab")
@@
 			)
 		)
-		(property "Value" "BC846"
+		(property "Value" "BC847"
 			(at 0 -2.4 90)
 			(layer "B.Fab")
@@
 			)
 		)
-		(property "Value" "AO3400A"
+		(property "Value" "BSS138"
 			(at 0 -2.4 90)
 			(layer "B.Fab")
@@
 			)
 		)
-		(property "Value" "AO3400A"
+		(property "Value" "BSS138"
 			(at 0 -2.4 0)
 			(layer "B.Fab")
@@
 			)
 		)
-		(property "Value" "AO3400A"
+		(property "Value" "BSS138"
 			(at 0 -2.4 90)
 			(layer "B.Fab")
@@
 			)
 		)
-		(property "Value" "R_Small"
+		(property "Value" "1k"
 			(at 0 -1.83 90)
 			(layer "B.Fab")
@@
 			)
 		)
-		(property "Value" "1u"
+		(property "Value" "100p"
 			(at 0 -1.85 90)
 			(layer "B.Fab")
@@
 			)
 		)
-		(property "Value" "AO3400A"
+		(property "Value" "BSS138"
 			(at 0 -2.4 0)
 			(layer "B.Fab")
@@
 			)
 		)
-		(property "Value" "C_Small"
+		(property "Value" "10u"
 			(at 0 -1.85 0)
 			(layer "B.Fab")
@@
 			)
 		)
-		(property "Value" "C_Small"
+		(property "Value" "100n"
 			(at 0 -1.85 0)
 			(layer "B.Fab")
@@
 			)
 		)
-		(property "Value" "10k"
+		(property "Value" "240k"
 			(at 0 -1.83 0)
 			(layer "B.Fab")
@@
 			)
 		)
-		(property "Value" "R_Small"
+		(property "Value" "1M"
 			(at 0 -1.83 0)
 			(layer "B.Fab")
@@
 			)
 		)
-		(property "Value" "R_Small"
+		(property "Value" "100k"
 			(at 0 -1.83 0)
 			(layer "B.Fab")
@@
 			)
 		)
-		(property "Value" "R_Small"
+		(property "Value" "100k"
 			(at 0 -1.83 0)
 			(layer "B.Fab")
@@
 			)
 		)
-		(property "Value" "R_Small"
+		(property "Value" "1M"
 			(at 0 -1.83 0)
 			(layer "B.Fab")
@@
 			)
 		)
-		(property "Value" "47k"
+		(property "Value" "470k"
 			(at 0 -1.83 90)
 			(layer "B.Fab")
